Commit message: Actualiza dimensiones del brazo RRR y refactoriza cinemática
URDF (robotRRR.urdf): l1 0.15→0.20 m, l2 0.30→0.35 m, l3 0.45→0.50 m.
Ajusta origins de juntas, centros visuales y comentarios en cadena.

kinematics.py: centraliza dimensiones (h, L1, L2) en el constructor en
lugar de repetirlas en fwd_kin e inv_kin. Extrae _quintic_profile y
_central_diff como helpers. Misma lógica y mismos nombres públicos;
verificado error=0 en 2000 muestras frente a implementación de referencia.

https://claude.ai/code/session_01GwJKPFuFEuDd6kUiJEPdcu

File: proyecto/Ros/proyecto_ws/src/robot_description/urdf/robotRRR.urdf (robot description, URDF)
Before this commit: robot robot_rrr, 5 links, 4 joints
Links:
- link arm_link: geometry visual box size=0.05 0.05 0.35
- link forearm_link: geometry visual box size=0.05 0.05 0.50
- link shoulder_link: geometry visual box size=0.05 0.05 0.20
Joints:
- joint arm_joint: origin xyz=0 0 0.15 rpy=0 0 0 -> xyz=0 0 0.20 rpy=0 0 0
- joint end_effector_joint: origin xyz=0 0 0.45 rpy=0 0 0 -> xyz=0 0 0.50 rpy=0 0 0
- joint forearm_joint: origin xyz=0 0 0.30 rpy=0 0 0 -> xyz=0 0 0.35 rpy=0 0 0
