Commit message: cambios actualizados (terminado)

File: proyecto/Ros/proyecto_ws/src/install/robot_description/share/robot_description/urdf/robotRRR.urdf (robot description, URDF)
Before this commit: robot robot_rrr, 4 links, 3 joints
Links:
- added link end_effector_link; visual sphere radius=0.04
- link arm_link: geometry visual box size=0.05 0.05 0.23
- link base_link: geometry visual cylinder length=0.05 radius=0.15
- link forearm_link: geometry visual box size=0.05 0.05 0.37
- link shoulder_link: geometry visual box size=0.05 0.05 0.17
Joints:
- added joint end_effector_joint: type fixed, parent forearm_link, child end_effector_link, origin xyz=0 0 0.37 rpy=0 0 0
- joint arm_joint: limit lower=-1.57 upper=1.57 effort=10 velocity=1 -> lower=-3.14 upper=3.14 effort=10 velocity=1; origin xyz=0 0 0.15 -> xyz=0 0 0.17 rpy=0 0 0
- joint forearm_joint: limit lower=-1.57 upper=1.57 effort=10 velocity=1 -> lower=-3.14 upper=3.14 effort=10 velocity=1; origin xyz=0 0 0.3 -> xyz=0 0 0.23 rpy=0 0 0
- joint shoulder_joint: origin xyz=0 0 0 -> xyz=0 0 0 rpy=0 0 0

File: proyecto/Ros/proyecto_ws/src/robot_description/urdf/robotRRR.urdf (robot description, URDF)
Before this commit: robot robot_rrr, 5 links, 4 joints
Links:
- link arm_link: geometry visual box size=0.05 0.05 0.23
- link base_link: geometry visual cylinder length=0.05 radius=0.15
- link end_effector_link: geometry visual sphere radius=0.04
- link forearm_link: geometry visual box size=0.05 0.05 0.37
- link shoulder_link: geometry visual box size=0.05 0.05 0.17
Joints:
- joint arm_joint: limit lower=-1.57 upper=1.57 effort=10 velocity=1 -> lower=-3.14 upper=3.14 effort=10 velocity=1; origin xyz=0 0 0.15 rpy=0 0 0 -> xyz=0 0 0.17 rpy=0 0 0
- joint end_effector_joint: origin xyz=0 0 0.45 rpy=0 0 0 -> xyz=0 0 0.37 rpy=0 0 0
- joint forearm_joint: limit lower=-1.57 upper=1.57 effort=10 velocity=1 -> lower=-3.14 upper=3.14 effort=10 velocity=1; origin xyz=0 0 0.30 rpy=0 0 0 -> xyz=0 0 0.23 rpy=0 0 0
